Commit message: Fix camera, robot spawn height, and add navigation launch files

File: my_robot/urdf/Assem2_pkg.urdf (robot description, URDF)
Before this commit: robot Assem2.SLDASM, 8 links, 7 joints
Links:
- added link camera_link, mass 0.1; collision box size=0.03 0.08 0.03; visual box size=0.03 0.08 0.03
- added link lidar_link, mass 0.2; collision cylinder length=0.06 radius=0.05; visual cylinder length=0.06 radius=0.05
- link back_leftwheel: geometry collision mesh filename=file:///home/nero/nero/my_robot/meshes/back_leftwheel.STL; visual mesh filename=file:///home/nero/nero/my_robot/meshes/back_leftwheel.STL
- link back_rigtwheel: geometry collision mesh filename=file:///home/nero/nero/my_robot/meshes/back_rigtwheel.STL; visual mesh filename=file:///home/nero/nero/my_robot/meshes/back_rigtwheel.STL
- link base_link: mass 14.5955135474013 -> 30.0; geometry collision mesh filename=file:///home/nero/nero/my_robot/meshes/base_link.STL; visual mesh filename=file:///home/nero/nero/my_robot/meshes/base_link.STL
- link front_leftwheel: geometry collision mesh filename=file:///home/nero/nero/my_robot/meshes/front_leftwheel.STL; visual mesh filename=file:///home/nero/nero/my_robot/meshes/front_leftwheel.STL
- link front_rightwheel: geometry collision mesh filename=file:///home/nero/nero/my_robot/meshes/front_rightwheel.STL; visual mesh filename=file:///home/nero/nero/my_robot/meshes/front_rightwheel.STL
- link leftarm: geometry collision mesh filename=file:///home/nero/nero/my_robot/meshes/leftarm.STL; visual mesh filename=file:///home/nero/nero/my_robot/meshes/leftarm.STL
- link rightarm: geometry collision mesh filename=file:///home/nero/nero/my_robot/meshes/rightarm.STL; visual mesh filename=file:///home/nero/nero/my_robot/meshes/rightarm.STL
Joints:
- added joint camera_joint: type fixed, parent base_link, child camera_link, origin xyz=0.15 0 0.25 rpy=0 0 0
- added joint lidar_joint: type fixed, parent base_link, child lidar_link, origin xyz=0 0 0.35 rpy=0 0 0
